File: AC Power Supply.kicad_pcb (KiCad board)
At the start: 2 copper layers, 81 x 37.4 mm, 56 parts, among them IC1 AMC1301DWVR, IC2 MCP6022T-E_SN, IC3 MCP1501T-20E_CHY, IC4 ATmega328-P, J1 Conn_01x16_Female, J2 Conn_01x02_Male, J3 Conn_01x02_Male, Y1 16MHz

Commit message: Revision 1.2.0
Parts:
- removed DS1: WC1602A, Display:WC1602A
- removed IC1: AMC1301DWVR, Package_SO:SOIC-8_7.5x5.85mm_P1.27mm
- removed IC2: MCP6022T-E_SN, Package_SO:SOIC-8_3.9x4.9mm_P1.27mm
- removed IC3: MCP1501T-20E_CHY, Package_TO_SOT_SMD:SOT-23-6_Handsoldering
- added J4: Conn_01x04_Male, Connector_PinHeader_2.54mm:PinHeader_1x04_P2.54mm_Vertical, F.Cu at (95.9, 67.8)
- added NT1: NetTie_2, NetTie:NetTie-2_THT_Pad0.3mm, F.Cu at (85.7, 77.4)
- added NT2: NetTie_2, NetTie:NetTie-2_THT_Pad0.3mm, F.Cu at (85.7, 76.0)
- added TP1: TestPoint, TestPoint:TestPoint_THTPad_D1.0mm_Drill0.5mm, F.Cu at (55.9, 75.7)
- added TP2: TestPoint, TestPoint:TestPoint_THTPad_D1.0mm_Drill0.5mm, F.Cu at (55.9, 78.7)
- added TP3: TestPoint, TestPoint:TestPoint_THTPad_D1.0mm_Drill0.5mm, F.Cu at (125.0, 73.6)
- added U1: MCP6022, Package_SO:SOIC-8_3.9x4.9mm_P1.27mm, F.Cu at (120.4, 69.6)
- added U2: MCP1501-20xCH, Package_TO_SOT_SMD:SOT-23-6_Handsoldering, F.Cu at (104.8, 73.3)
- added U3: AMC1301DWVR, AMC1301DWVR:AMC1301DWVR, F.Cu at (71.9, 76.7)
- C12: value 2.2uF -> 1nF
- H1, H2, H3, H4: footprint MountingHole:MountingHole_2.7mm_M2.5_DIN965_Pad -> MountingHole:MountingHole_2.7mm_M2.5_DIN965
- J2, J3: value Conn_01x02_Male -> B2B-XH-A(LF)(SN); footprint Connector_PinHeader_2.54mm:PinHeader_1x02_P2.54mm_Vertical -> B2B-XH-A_LF__SN_:JST_B2B-XH-A(LF)(SN)
- L1: value L -> 10uH
- R18: value 10 -> 10k
- RV1: footprint Potentiometer_SMD:Potentiometer_Bourns_3214X_Vertical -> 64WR10KLF:64WR10KLF
- moved J2 72.1 mm to (54.0, 60.6)
- moved J3 29.2 mm to (77.5, 52.4), turned to 90 degrees
- moved R13 25.0 mm to (114.5, 74.2), turned to 180 degrees
- moved C8 25.0 mm to (114.5, 72.0), turned to 180 degrees
- moved R16 24.8 mm to (126.1, 71.4), turned to 180 degrees
- moved C18 24.3 mm to (83.4, 62.1), turned to -90 degrees
- moved C10 23.9 mm to (126.1, 67.9)
- moved C14 22.9 mm to (100.0, 73.3), turned to 0 degrees
- moved C7 21.2 mm to (116.7, 77.7)
- moved R14 20.3 mm to (113.6, 76.8), turned to 180 degrees
- moved R10 19.0 mm to (97.3, 78.6)
- moved R12 19.0 mm to (104.1, 78.6)
- moved locked 18.9 mm to (100.8, 77.5), turned to -90 degrees
- moved R11 18.7 mm to (104.1, 76.4)
- moved R9 18.7 mm to (97.3, 76.4)
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- renumbered C6 to locked, J1 to locked
Connections:
- C1 pad 1: /VDC1 -> /GND1
- C1 pad 2: /GND1 -> /VDC1
- C10 pad 1: VDC -> GND
- C10 pad 2: GND -> VDC
- C2 pad 1: /VDC1 -> /GND1
- C2 pad 2: /GND1 -> /VDC1
- J2 pad 1: VDC -> VIN2
- J2 pad 2: GND -> VIN1
- J3 pad 1: VIN1 -> VDC
- J3 pad 2: VIN2 -> GND
- R8 pad 1: /VDC1 -> /GND1
- R8 pad 2: /GND1 -> /VDC1
Routing:
- net /GND1: track 0.00 -> 29.7 mm, vias 0 -> 1
- net AREF: track 7.63 -> 28.1 mm
- net GND: track 2.70 -> 18.5 mm, vias 14 -> 16
- net Net-(C18-Pad1): track 12.5 -> 23.7 mm
- net Net-(NT2-Pad2): track 3.36 -> 14.2 mm
- net Net-(C9-Pad2): track 9.94 -> 20.6 mm
- net Net-(NT1-Pad1): track 0.00 -> 8.76 mm
- net Net-(NT2-Pad1): track 0.00 -> 8.71 mm
- net Net-(R5-Pad2): track 7.29 -> 15.6 mm
- net Net-(R17-Pad1): track 9.84 -> 17.7 mm, vias 0 -> 2
- net Net-(C8-Pad1): track 25.8 -> 18.4 mm
- net /VDC1: track 13.2 -> 20.4 mm
- net VIN1: track 12.4 -> 6.51 mm
- net Net-(NT1-Pad2): track 4.08 -> 9.84 mm
- net Net-(IC4-Pad11): track 17.6 -> 12.0 mm
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Other:
- outline, holes or cut-outs redrawn
- board text added: "+5V"
- board text added: "A0"
- board text added: "AC Voltmeter"
- board text added: "AREF"
- board text added: "GND"
- board text added: "Revision 1.2.0"
- board text added: "VIN1"
- board text added: "VIN2"
- board text added: "© 2022 Nikolaj Brinch Jørgensen"
