File: AC Power Supply.kicad_sch (KiCad schematic)
At the start: 56 parts, among them IC1 AMC1301DWVR, IC2 MCP6022T-E_SN, IC3 MCP1501T-20E_CHY, IC4 ATmega328-P, J1 Conn_01x16_Female, J2 Conn_01x02_Male, J3 Conn_01x02_Male, Y1 16MHz

Commit message: Revision 1.2.0
Parts:
- removed DS1: WC1602A, Display:WC1602A, symbol Display_Character:WC1602A
- removed IC1: AMC1301DWVR, Package_SO:SOIC-8_7.5x5.85mm_P1.27mm, symbol AMC1301DWVR:AMC1301DWVR
- removed IC2: MCP6022T-E_SN, Package_SO:SOIC-8_3.9x4.9mm_P1.27mm, symbol MCP6022T-E_SN:MCP6022T-E_SN
- removed IC3: MCP1501T-20E_CHY, Package_TO_SOT_SMD:SOT-23-6_Handsoldering, symbol MCP1501T-20E_CHY:MCP1501T-20E_CHY
- removed J2, J3: Conn_01x02_Male, Connector_PinHeader_2.54mm:PinHeader_1x02_P2.54mm_Vertical, symbol Connector:Conn_01x02_Male
- added J2, J3: B2B-XH-A(LF)(SN), B2B-XH-A_LF__SN_:JST_B2B-XH-A(LF)(SN), symbol B2B-XH-A_LF__SN_:B2B-XH-A(LF)(SN)
- added J4: Conn_01x04_Male, Connector_PinHeader_2.54mm:PinHeader_1x04_P2.54mm_Vertical, symbol Connector:Conn_01x04_Male
- added NT1, NT2: NetTie_2, NetTie:NetTie-2_THT_Pad0.3mm, symbol Device:NetTie_2
- added TP1, TP2, TP3: TestPoint, TestPoint:TestPoint_THTPad_D1.0mm_Drill0.5mm, symbol Connector:TestPoint
- added U1: MCP6022, Package_SO:SOIC-8_3.9x4.9mm_P1.27mm, symbol Amplifier_Operational:MCP6022
- added U2: MCP1501-20xCH, Package_TO_SOT_SMD:SOT-23-6_Handsoldering, symbol Reference_Voltage:MCP1501-20xCH
- added U3: AMC1301DWVR, AMC1301DWVR:AMC1301DWVR, symbol Amplifier_Difference:AMC1300DWV
- C12: value 2.2uF -> 1nF
- H1, H2, H3, H4: footprint MountingHole:MountingHole_2.7mm_M2.5_DIN965_Pad -> MountingHole:MountingHole_2.7mm_M2.5_DIN965; symbol Mechanical:MountingHole_Pad -> Mechanical:MountingHole
- R18: value 10 -> 10k
- RV1: footprint Potentiometer_SMD:Potentiometer_Bourns_3214X_Vertical -> 64WR10KLF:64WR10KLF; symbol Device:R_Potentiometer_Trim -> 64WR10KLF:64WR10KLF
Connections:
- net A0: now also J4.2 (Pin_2)
- net AREF: now also J4.1 (Pin_1)
- net GND: now also C10.1, J3.2, J4.4 (Pin_4), U1.4 (V-), U2.2 (GND), U2.3 (GND), U2.5 (GND), U3.5 (V-); no longer C10.2, H1.1, H2.1, H3.1, H4.1
- net GND1: now also C1.1, C2.1, R8.1, TP2.1, U3.3 (-), U3.4 (V-); no longer C1.2, C2.2, R8.2
- net VDC: now also C10.2, J3.1, J4.3 (Pin_3), U1.8 (V+), U2.4 (~{SHDN}), U2.6 (VDD), U3.8 (V+); no longer C10.1
- net VDC1: now also C1.2, C2.2, R8.2, U3.1 (V+); no longer C1.1, C2.1, R8.1
- net VIN1: now also J2.2
- net VIN2: now also J2.1
- net at R17.1, R19.1, R20.1: now also U2.1 (OUT)
- net at C8.1, R11.2, R13.1: now also U1.2 (-)
- net at C8.2, R13.2, R15.1: now also U1.1
- net at R16.2: now also TP3.1, U1.6 (-), U1.7
- net at C7.1, R12.2, R14.2: now also U1.3 (+)
- net at C12.1, R17.2, R18.1: now also U1.5 (+)
- net at R9.1: now also NT1.2
- net at R5.2, R7.2: now also TP1.1, U3.2 (+)
- net at R10.1: now also NT2.2
- new net: NT2.1, U3.7 (+)
- new net: NT1.1, U3.6 (-)
Other:
- moved on the sheet: C1, C10, C12, C13, C14, C2, C3, C4, C5, C6, C7, C8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
